Commit message: Update

File: install/flembot_description/share/flembot_description/urdf/flembot.urdf.xacro (robot description, xacro)
@@ -1 +1,10 @@
-/home/vboxuser/ros2_ws/src/flembot_description/urdf/flembot.urdf.xacro
+<?xml version="1.0"?>
+<robot xmlns:xacro="http://ros.org/wiki/xacro" name="flembot">
+  <link name="base_link">
+    <visual>
+      <geometry>
+        <box size="0.3 0.3 0.1"/>
+      </geometry>
+    </visual>
+  </link>
+</robot>
